File: Hardware/SmartInsole_Right/SmartInsole_Right/SmartInsole_Right.kicad_pcb (KiCad board)
At the start: 2 copper layers, 49.4 x 29.7 mm, 106 parts, among them IC1 MIC5225-1.8YM5-TR, J1 USB_C_Receptacle_USB2.0, J2 1769, J3 200528-0200 PI, Q1 BSS138, Q2 BSS138, Q3 BSS138, Q4 BSS138, Q5 DMG3415U, Q7 IRF7343PBF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

Commit message: feat: change component position
Parts:
- U4: moved to B.Cu
- moved R25 24.4 mm to (127.0, 121.4), turned to 90 degrees
- moved R23 24.3 mm to (127.1, 117.6), turned to 90 degrees
- moved JP1 23.2 mm to (127.3, 114.2), turned to 90 degrees
- moved R30 22.4 mm to (135.6, 126.6)
- moved C8 22.4 mm to (135.7, 124.6)
- moved R28 21.4 mm to (129.7, 114.2), turned to -90 degrees
- moved D3 19.8 mm to (156.8, 142.0)
- moved U4 19.8 mm to (122.9, 117.9), turned to 0 degrees
- moved C1 17.1 mm to (135.7, 122.7), turned to 0 degrees
- moved C10 16.7 mm to (135.7, 116.9)
- moved C9 16.7 mm to (135.7, 118.8)
- moved C4 16.6 mm to (135.7, 120.8), turned to 0 degrees
- moved R38 9.02 mm to (152.3, 140.8)
- moved D1 8.17 mm to (127.2, 110.7), turned to -90 degrees
- moved R29 7.26 mm to (135.7, 114.2)
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Connections:
- Q1 pad 3: /SDI/SDA -> /SDA
- Q2 pad 3: /SCK/SCL -> /SCL
- R23 pad 1: /SDI/SDA -> /SDA
- R25 pad 1: /SCK/SCL -> /SCL
Routing:
- net +1V8: track 6.04 -> 31.5 mm
- net GND: track 162.0 -> 177.3 mm
- net +3V3: track 44.2 -> 50.4 mm
- net /INT: track 1.80 -> 6.73 mm
- net /SDO/ADR: track 1.84 -> 4.95 mm
- net /SCL: track 19.4 -> 22.0 mm
- net /SDA: track 20.2 -> 22.7 mm
- net /INT_1.8V: track 0.00 -> 2.03 mm
- net /CS_1.8V: track 0.00 -> 1.99 mm
- net /Vref: track 0.00 -> 1.92 mm
- net /SDI/SDA: track 1.81 -> 0.00 mm
- net /SCK/SCL: track 1.81 -> 0.00 mm

Commit message: feat: added 3D
Parts:
- moved R14 16.9 mm to (147.9, 113.2)
- moved R17 16.9 mm to (143.7, 113.3)
- moved C5 16.9 mm to (155.4, 109.1)
- moved C6 16.9 mm to (155.7, 111.3)
- moved R11 16.9 mm to (156.3, 104.7)
- moved R12 16.9 mm to (156.3, 106.6)
- moved R15 16.9 mm to (143.7, 117.3)
- moved R16 16.9 mm to (143.7, 115.3)
- moved R19 16.9 mm to (156.4, 115.2)
- moved R2 16.9 mm to (143.7, 121.2)
- moved R20 16.9 mm to (156.4, 117.2)
- moved R21 16.9 mm to (156.4, 119.2)
- moved R22 16.9 mm to (143.7, 119.2)
- moved R3 16.9 mm to (151.8, 109.0)
- moved R4 16.9 mm to (147.9, 109.0)
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
Commit message: feat: added more libraries
Parts:
- IC1: footprint MIC5225-1.8YM5-TR:SOT95P280X130-5N -> Regulador_MIC5225-1.8YM5-TR:SOT95P280X130-5N
- J2: footprint JST_PH_2:1769 -> ConectorBateria_JST_PH:1769
- J3: footprint 200528-0200:2005280200 -> ConectorSensores_200528-0200:2005280200
- RN1, RN2, RN3, RN4: footprint TC164-FR-07270KL:RESCAV80P320X160X70-8N -> ResistorPack_C164-FR-07270KL:RESCAV80P320X160X70-8N
- S1, S3: footprint KMR211NGLFS:SW_KMR211NGLFS -> Pulsador_KMR211:SW_KMR211NGLFS
- U7: footprint CP2102N-A02-GQFN24R:QFN50P400X400X80-25N -> USB_Serial_CP2102N:QFN50P400X400X80-25N
