File: Hardware/SmartInsole_Right/SmartInsole_Right/SmartInsole_Right.kicad_sch (KiCad schematic)
At the start: 107 parts, among them IC1 MIC5225-1.8YM5-TR, J1 USB_C_Receptacle_USB2.0, J2 1769, J3 200528-0200 PI, Q1 BSS138, Q2 BSS138, Q3 BSS138, Q4 BSS138, Q5 DMG3415U, Q6 DUAL NPN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

Commit message: feat: Added component libraries
Parts:
- D3: footprint NeoPixel_2758:SOL320P540X170-4N -> NeoPixel_2758_FP:SOL320P540X170-4N
- IC1: footprint SOT95P280X130-5N -> MIC5225-1.8YM5-TR_FP:SOT95P280X130-5N
- J3: footprint 2005280200 -> 200528-0200_FP:2005280200
- RN1, RN2, RN3, RN4: footprint TC164-FR-07270KL:RESCAV80P320X160X70-8N -> C164-FR-07270KL_FP:RESCAV80P320X160X70-8N
- S1, S3: footprint KMR211NGLFS:SW_KMR211NGLFS -> KMR211NGLFS_FP:SW_KMR211NGLFS
- U7: footprint CP2102N-A02-GQFN24R:QFN50P400X400X80-25N -> CP2102N_FP:QFN50P400X400X80-25N
Connections:
- net SCK/SCL is gone; now on net SCL: Q2.3 (D), R25.1
- net SDI/SDA is gone; now on net SDA: Q1.3 (D), R23.1
Changed lines of the file:
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@@
     (effects (font (size 1.27 1.27)) (justify right bottom))
   )
-  (label "SDI{slash}SDA" (at 294.894 161.29 180) (fields_autoplaced)
+  (label "SDA" (at 294.894 161.29 180) (fields_autoplaced)
     (effects (font (size 1.27 1.27)) (justify right bottom))
   )
@@
     (effects (font (size 1.27 1.27)) (justify right bottom))
   )
-  (label "SCK{slash}SCL" (at 294.894 189.738 180) (fields_autoplaced)
+  (label "SCL" (at 294.894 189.738 180) (fields_autoplaced)
     (effects (font (size 1.27 1.27)) (justify right bottom))
   )
@@
       (effects (font (size 1.27 1.27)))
     )
-    (property "Footprint" "TC164-FR-07270KL:RESCAV80P320X160X70-8N" (at 139.954 192.278 0)
+    (property "Footprint" "C164-FR-07270KL_FP:RESCAV80P320X160X70-8N" (at 139.954 192.278 0)
       (effects (font (size 1.27 1.27)) (justify bottom) hide)
     )
@@
       (effects (font (size 1.27 1.27)))
     )
-    (property "Footprint" "CP2102N-A02-GQFN24R:QFN50P400X400X80-25N" (at 358.394 49.784 0)
+    (property "Footprint" "CP2102N_FP:QFN50P400X400X80-25N" (at 358.394 49.784 0)
       (effects (font (size 1.27 1.27)) (justify bottom) hide)
     )
@@
       (effects (font (size 1.27 1.27)))
     )
-    (property "Footprint" "TC164-FR-07270KL:RESCAV80P320X160X70-8N" (at 139.7 226.06 0)
+    (property "Footprint" "C164-FR-07270KL_FP:RESCAV80P320X160X70-8N" (at 139.7 226.06 0)
       (effects (font (size 1.27 1.27)) (justify bottom) hide)
     )
@@
       (effects (font (size 1.27 1.27)))
     )
-    (property "Footprint" "TC164-FR-07270KL:RESCAV80P320X160X70-8N" (at 96.266 192.278 0)
+    (property "Footprint" "C164-FR-07270KL_FP:RESCAV80P320X160X70-8N" (at 96.266 192.278 0)
       (effects (font (size 1.27 1.27)) (justify bottom) hide)
     )
@@
       (effects (font (size 1.27 1.27)) (justify right))
     )
-    (property "Footprint" "KMR211NGLFS:SW_KMR211NGLFS" (at 119.126 110.236 0)
+    (property "Footprint" "KMR211NGLFS_FP:SW_KMR211NGLFS" (at 119.126 110.236 0)
       (effects (font (size 1.27 1.27)) (justify bottom) hide)
     )
@@
       (effects (font (size 1.27 1.27)))
     )
-    (property "Footprint" "SOT95P280X130-5N" (at 312.166 199.06 0)
+    (property "Footprint" "MIC5225-1.8YM5-TR_FP:SOT95P280X130-5N" (at 312.166 199.06 0)
       (effects (font (size 1.27 1.27)) (justify left top) hide)
     )
@@
       (effects (font (size 1.27 1.27)))
     )
-    (property "Footprint" "2005280200" (at 40.386 277.8 0)
+    (property "Footprint" "200528-0200_FP:2005280200" (at 40.386 277.8 0)
       (effects (font (size 1.27 1.27)) (justify left top) hide)
     )
@@
       (effects (font (size 1.27 1.27)))
     )
-    (property "Footprint" "NeoPixel_2758:SOL320P540X170-4N" (at 84.074 93.726 0)
+    (property "Footprint" "NeoPixel_2758_FP:SOL320P540X170-4N" (at 84.074 93.726 0)
       (effects (font (size 1.27 1.27)) (justify bottom) hide)
     )
@@
       (effects (font (size 1.27 1.27)))
     )
-    (property "Footprint" "TC164-FR-07270KL:RESCAV80P320X160X70-8N" (at 96.774 224.79 0)
+    (property "Footprint" "C164-FR-07270KL_FP:RESCAV80P320X160X70-8N" (at 96.774 224.79 0)
       (effects (font (size 1.27 1.27)) (justify bottom) hide)
     )
@@
       (effects (font (size 1.27 1.27)) (justify right))
     )
-    (property "Footprint" "KMR211NGLFS:SW_KMR211NGLFS" (at 240.03 52.832 0)
+    (property "Footprint" "KMR211NGLFS_FP:SW_KMR211NGLFS" (at 240.03 52.832 0)
       (effects (font (size 1.27 1.27)) (justify bottom) hide)
     )

Commit message: feat: added more libraries
Parts:
- D3: footprint NeoPixel_2758_FP:SOL320P540X170-4N -> NeoPixel_2758:SOL320P540X170-4N
- IC1: footprint MIC5225-1.8YM5-TR_FP:SOT95P280X130-5N -> Regulador_MIC5225-1.8YM5-TR:SOT95P280X130-5N
- J2: footprint JST_PH_2:1769 -> ConectorBateria_JST_PH:1769
- J3: footprint 200528-0200_FP:2005280200 -> ConectorSensores_200528-0200:2005280200
- RN1, RN2, RN3, RN4: footprint C164-FR-07270KL_FP:RESCAV80P320X160X70-8N -> ResistorPack_C164-FR-07270KL:RESCAV80P320X160X70-8N
- S1, S3: footprint KMR211NGLFS_FP:SW_KMR211NGLFS -> Pulsador_KMR211:SW_KMR211NGLFS
- U7: footprint CP2102N_FP:QFN50P400X400X80-25N -> USB_Serial_CP2102N:QFN50P400X400X80-25N
Changed lines of the file:
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@@
       (effects (font (size 1.27 1.27)))
     )
-    (property "Footprint" "C164-FR-07270KL_FP:RESCAV80P320X160X70-8N" (at 139.954 192.278 0)
+    (property "Footprint" "ResistorPack_C164-FR-07270KL:RESCAV80P320X160X70-8N" (at 139.954 192.278 0)
       (effects (font (size 1.27 1.27)) (justify bottom) hide)
     )
@@
       (effects (font (size 1.27 1.27)))
     )
-    (property "Footprint" "CP2102N_FP:QFN50P400X400X80-25N" (at 358.394 49.784 0)
+    (property "Footprint" "USB_Serial_CP2102N:QFN50P400X400X80-25N" (at 358.394 49.784 0)
       (effects (font (size 1.27 1.27)) (justify bottom) hide)
     )
@@
       (effects (font (size 1.27 1.27)))
     )
-    (property "Footprint" "C164-FR-07270KL_FP:RESCAV80P320X160X70-8N" (at 139.7 226.06 0)
+    (property "Footprint" "ResistorPack_C164-FR-07270KL:RESCAV80P320X160X70-8N" (at 139.7 226.06 0)
       (effects (font (size 1.27 1.27)) (justify bottom) hide)
     )
@@
       (effects (font (size 1.27 1.27)))
     )
-    (property "Footprint" "JST_PH_2:1769" (at 109.22 157.658 0)
+    (property "Footprint" "ConectorBateria_JST_PH:1769" (at 109.22 157.658 0)
       (effects (font (size 1.27 1.27)) (justify left top) hide)
     )
@@
       (effects (font (size 1.27 1.27)))
     )
-    (property "Footprint" "C164-FR-07270KL_FP:RESCAV80P320X160X70-8N" (at 96.266 192.278 0)
+    (property "Footprint" "ResistorPack_C164-FR-07270KL:RESCAV80P320X160X70-8N" (at 96.266 192.278 0)
       (effects (font (size 1.27 1.27)) (justify bottom) hide)
     )
@@
       (effects (font (size 1.27 1.27)) (justify right))
     )
-    (property "Footprint" "KMR211NGLFS_FP:SW_KMR211NGLFS" (at 119.126 110.236 0)
+    (property "Footprint" "Pulsador_KMR211:SW_KMR211NGLFS" (at 119.126 110.236 0)
       (effects (font (size 1.27 1.27)) (justify bottom) hide)
     )
@@
       (effects (font (size 1.27 1.27)))
     )
-    (property "Footprint" "MIC5225-1.8YM5-TR_FP:SOT95P280X130-5N" (at 312.166 199.06 0)
+    (property "Footprint" "Regulador_MIC5225-1.8YM5-TR:SOT95P280X130-5N" (at 312.166 199.06 0)
       (effects (font (size 1.27 1.27)) (justify left top) hide)
     )
@@
       (effects (font (size 1.27 1.27)))
     )
-    (property "Footprint" "200528-0200_FP:2005280200" (at 40.386 277.8 0)
+    (property "Footprint" "ConectorSensores_200528-0200:2005280200" (at 40.386 277.8 0)
       (effects (font (size 1.27 1.27)) (justify left top) hide)
     )
@@
       (effects (font (size 1.27 1.27)))
     )
-    (property "Footprint" "NeoPixel_2758_FP:SOL320P540X170-4N" (at 84.074 93.726 0)
+    (property "Footprint" "NeoPixel_2758:SOL320P540X170-4N" (at 84.074 93.726 0)
       (effects (font (size 1.27 1.27)) (justify bottom) hide)
     )
@@
       (effects (font (size 1.27 1.27)))
     )
-    (property "Footprint" "C164-FR-07270KL_FP:RESCAV80P320X160X70-8N" (at 96.774 224.79 0)
+    (property "Footprint" "ResistorPack_C164-FR-07270KL:RESCAV80P320X160X70-8N" (at 96.774 224.79 0)
       (effects (font (size 1.27 1.27)) (justify bottom) hide)
     )
@@
       (effects (font (size 1.27 1.27)) (justify right))
     )
-    (property "Footprint" "KMR211NGLFS_FP:SW_KMR211NGLFS" (at 240.03 52.832 0)
+    (property "Footprint" "Pulsador_KMR211:SW_KMR211NGLFS" (at 240.03 52.832 0)
       (effects (font (size 1.27 1.27)) (justify bottom) hide)
     )
